File: audio.kicad_sch (KiCad schematic)
At the start: 34 parts, among them J2 Audio Jack, J5 Speaker, U6 UDA1334ATS, U7 PAM8403D

Commit message: revA3
Parts:
- U6: footprint Package_SO:SSOP-16_4.4x5.2mm_P0.65mm -> footprints:SSOP-16_4.4x5.2mm_P0.65mm-extended
Changed lines of the file:
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@@
 	(title_block
 		(title "Karabas Esplay")
-		(date "2025-09-30")
-		(rev "A2")
+		(date "2025-10-04")
+		(rev "A3")
 		(company "Andy Karpov production")
 	)
@@
 			)
 		)
-		(property "Footprint" "Package_SO:SSOP-16_4.4x5.2mm_P0.65mm"
+		(property "Footprint" "footprints:SSOP-16_4.4x5.2mm_P0.65mm-extended"
 			(at 97.79 76.2 0)
 			(effects
