File: autofire.kicad_sch (KiCad schematic)
At the start: 14 parts, among them SW14 C, SW15 D, U10 LMC555xM, U9 LMC555xM

Commit message: Added revA2
Parts:
- SW14, SW15: footprint Button_Switch_SMD:SW_Push_1TS009xxxx-xxxx-xxxx_6x6x5mm -> footprints:SW_Push_1TS009_combined1
Changed lines of the file:
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@@
 	(title_block
 		(title "Karabas Esplay")
-		(date "2025-09-28")
-		(rev "A")
+		(date "2025-09-30")
+		(rev "A2")
 		(company "Andy Karpov production")
 	)
@@
 			)
 		)
-		(property "Footprint" "Button_Switch_SMD:SW_Push_1TS009xxxx-xxxx-xxxx_6x6x5mm"
+		(property "Footprint" "footprints:SW_Push_1TS009_combined1"
 			(at 128.27 59.69 0)
 			(effects
@@
 			)
 		)
-		(property "Footprint" "Button_Switch_SMD:SW_Push_1TS009xxxx-xxxx-xxxx_6x6x5mm"
+		(property "Footprint" "footprints:SW_Push_1TS009_combined1"
 			(at 57.15 59.69 0)
 			(effects
