File: mcu.kicad_sch (KiCad schematic)
At the start: 70 parts, among them J1 USB_C_Receptacle_USB2.0_16P, J3 ILI9341 3.2", J4 Battery, Q1 MMBT2222A, Q2 MMBT2222A, Q3 MMBT2222A, Q4 IRLML6402, SW1 Reset, SW10 L_BTN, SW11 MENU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

Commit message: Final revA
Parts:
- added BAT+1: +, TestPoint:TestPoint_Pad_D3.0mm, symbol Connector:TestPoint
- added BAT-1: -, TestPoint:TestPoint_Pad_D3.0mm, symbol Connector:TestPoint
- J4: footprint Connector_JST:JST_PH_S2B-PH-SM4-TB_1x02-1MP_P2.00mm_Horizontal -> Connector_JST:JST_PH_S2B-PH-K_1x02_P2.00mm_Horizontal
Connections:
- net GND: now also J4.2, BAT-1.1; no longer J4.1
- net V_BATT: now also J4.1, BAT+1.1; no longer J4.2

Commit message: Added revA2
Parts:
- SW11, SW2, SW3, SW4, SW5, SW6, SW7, SW8, SW9: footprint Button_Switch_SMD:SW_Push_1TS009xxxx-xxxx-xxxx_6x6x5mm -> footprints:SW_Push_1TS009_combined1
Changed lines of the file:
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@@
 	(title_block
 		(title "Karabas Esplay")
-		(date "2025-09-28")
-		(rev "A")
+		(date "2025-09-30")
+		(rev "A2")
 		(company "Andy Karpov production")
 	)
@@
 			)
 		)
-		(property "Footprint" "Button_Switch_SMD:SW_Push_1TS009xxxx-xxxx-xxxx_6x6x5mm"
+		(property "Footprint" "footprints:SW_Push_1TS009_combined1"
 			(at 214.63 99.06 0)
 			(effects
@@
 			)
 		)
-		(property "Footprint" "Button_Switch_SMD:SW_Push_1TS009xxxx-xxxx-xxxx_6x6x5mm"
+		(property "Footprint" "footprints:SW_Push_1TS009_combined1"
 			(at 167.64 99.06 0)
 			(effects
@@
 			)
 		)
-		(property "Footprint" "Button_Switch_SMD:SW_Push_1TS009xxxx-xxxx-xxxx_6x6x5mm"
+		(property "Footprint" "footprints:SW_Push_1TS009_combined1"
 			(at 149.86 99.06 0)
 			(effects
@@
 			)
 		)
-		(property "Footprint" "Button_Switch_SMD:SW_Push_1TS009xxxx-xxxx-xxxx_6x6x5mm"
+		(property "Footprint" "footprints:SW_Push_1TS009_combined1"
 			(at 158.75 99.06 0)
 			(effects
@@
 			)
 		)
-		(property "Footprint" "Button_Switch_SMD:SW_Push_1TS009xxxx-xxxx-xxxx_6x6x5mm"
+		(property "Footprint" "footprints:SW_Push_1TS009_combined1"
 			(at 140.97 99.06 0)
 			(effects
@@
 			)
 		)
-		(property "Footprint" "Button_Switch_SMD:SW_Push_1TS009xxxx-xxxx-xxxx_6x6x5mm"
+		(property "Footprint" "footprints:SW_Push_1TS009_combined1"
 			(at 132.08 99.06 0)
 			(effects
@@
 			)
 		)
-		(property "Footprint" "Button_Switch_SMD:SW_Push_1TS009xxxx-xxxx-xxxx_6x6x5mm"
+		(property "Footprint" "footprints:SW_Push_1TS009_combined1"
 			(at 194.31 99.06 0)
 			(effects
@@
 			)
 		)
-		(property "Footprint" "Button_Switch_SMD:SW_Push_1TS009xxxx-xxxx-xxxx_6x6x5mm"
+		(property "Footprint" "footprints:SW_Push_1TS009_combined1"
 			(at 176.53 99.06 0)
 			(effects
@@
 			)
 		)
-		(property "Footprint" "Button_Switch_SMD:SW_Push_1TS009xxxx-xxxx-xxxx_6x6x5mm"
+		(property "Footprint" "footprints:SW_Push_1TS009_combined1"
 			(at 185.42 99.06 0)
 			(effects
